File: HCKeyboard/HCKeyboard.kicad_pcb (KiCad board)
At the start: 2 copper layers, 338.1 x 128.6 mm, 161 parts, among them SW1 SW_Push, SW10 SW_Push, SW11 SW_Push, SW12 SW_Push, SW13 SW_Push, SW14 SW_Push, SW16 SW_Push, SW17 SW_Push, SW18 SW_Push, SW19 SW_Push, SW2 SW_Push, SW20 SW_Push, SW21 SW_Push, SW22 SW_Push, SW23 SW_Push, SW24 SW_Push, SW25 SW_Push, SW26 SW_Push, SW27 SW_Push, SW28 SW_Push, SW29 SW_Push, SW3 SW_Push, SW30 SW_Push, SW31 SW_Push, SW32 SW_Push, SW33 SW_Push, SW34 SW_Push, SW35 SW_Push, SW36 SW_Push, SW37 SW_Push, SW38 SW_Push, SW39 SW_Push, SW4 SW_Push, SW40 SW_Push, SW41 SW_Push, SW42 SW_Push, SW43 SW_Push, SW44 SW_Push, SW45 SW_Push, SW46 SW_Push, SW47 SW_Push, SW48 SW_Push, SW49 SW_Push, SW5 SW_Push, SW50 SW_Push, SW51 SW_Push, SW52 SW_Push, SW53 SW_Push, SW54 SW_Push, SW55 SW_Push, SW56 SW_Push, SW57 SW_Push, SW58 SW_Push, SW59 SW_Push, SW6 SW_Push, SW60 SW_Push, SW61 SW_Push, SW62 SW_Push, SW63 SW_Push, SW64 SW_Push, SW65 SW_Push, SW66 SW_Push, SW67 SW_Push, SW68 SW_Push, SW69 SW_Push, SW7 SW_Push, SW70 SW_Push, SW71 SW_Push, SW72 SW_Push, SW73 SW_Push, SW74 SW_Push, SW75 SW_Push, SW76 SW_Push, SW77 SW_Push, SW78 SW_Push, SW79 SW_Push, SW8 SW_Push, SW9 SW_Push

Commit message: PCB done! Exported files will be in the next commit.
Parts:
- moved D57 30.6 mm to (68.1, 128.6)
- moved A1 6.62 mm to (329.7, 26.4)
- moved D43 5.08 mm to (309.9, 90.5)
Routing:
- net /ROW5: track 0.00 -> 445.4 mm
- net /ROW4: track 0.00 -> 375.6 mm
- net /ROW3: track 0.00 -> 335.6 mm
- net /ROW2: track 0.00 -> 326.0 mm
- net /COL0: track 108.9 -> 423.7 mm
- net /ROW0: track 0.00 -> 297.7 mm
- net /COL1: track 119.7 -> 412.2 mm
- net /COL2: track 116.8 -> 394.7 mm
- net /ROW1: track 46.9 -> 312.8 mm
- net /COL3: track 92.8 -> 353.5 mm
- net /COL4: track 92.8 -> 338.8 mm
- net /COL5: track 115.8 -> 339.5 mm
- net /COL6: track 94.8 -> 301.6 mm
- net /COL12: track 163.9 -> 316.8 mm
- net /COL11: track 176.8 -> 326.2 mm
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- added copper zone on B.Cu, net Net-(A1-GND-Pad13)
- added copper zone on F.Cu, net Net-(A1-GND-Pad13)
Other:
- board size 338.1 x 128.6 mm -> 338.1 x 133.3 mm
