File: HCKeyboard/HCKeyboard.kicad_pcb (KiCad board)
At the start: 2 copper layers, 338.1 x 133.3 mm, 161 parts, among them SW1 SW_Push, SW10 SW_Push, SW11 SW_Push, SW12 SW_Push, SW13 SW_Push, SW14 SW_Push, SW16 SW_Push, SW17 SW_Push, SW18 SW_Push, SW19 SW_Push, SW2 SW_Push, SW20 SW_Push, SW21 SW_Push, SW22 SW_Push, SW23 SW_Push, SW24 SW_Push, SW25 SW_Push, SW26 SW_Push, SW27 SW_Push, SW28 SW_Push, SW29 SW_Push, SW3 SW_Push, SW30 SW_Push, SW31 SW_Push, SW32 SW_Push, SW33 SW_Push, SW34 SW_Push, SW35 SW_Push, SW36 SW_Push, SW37 SW_Push, SW38 SW_Push, SW39 SW_Push, SW4 SW_Push, SW40 SW_Push, SW41 SW_Push, SW42 SW_Push, SW43 SW_Push, SW44 SW_Push, SW45 SW_Push, SW46 SW_Push, SW47 SW_Push, SW48 SW_Push, SW49 SW_Push, SW5 SW_Push, SW50 SW_Push, SW51 SW_Push, SW52 SW_Push, SW53 SW_Push, SW54 SW_Push, SW55 SW_Push, SW56 SW_Push, SW57 SW_Push, SW58 SW_Push, SW59 SW_Push, SW6 SW_Push, SW60 SW_Push, SW61 SW_Push, SW62 SW_Push, SW63 SW_Push, SW64 SW_Push, SW65 SW_Push, SW66 SW_Push, SW67 SW_Push, SW68 SW_Push, SW69 SW_Push, SW7 SW_Push, SW70 SW_Push, SW71 SW_Push, SW72 SW_Push, SW73 SW_Push, SW74 SW_Push, SW75 SW_Push, SW76 SW_Push, SW77 SW_Push, SW78 SW_Push, SW79 SW_Push, SW8 SW_Push, SW9 SW_Push

Commit message: Added mounting holes.
Parts:
- added H1: MountingHole, MountingHole:MountingHole_3.2mm_M3, F.Cu at (29.8, 29.8)
- added H2: MountingHole, MountingHole:MountingHole_3.2mm_M3, F.Cu at (356.0, 29.8)
- added H3: MountingHole, MountingHole:MountingHole_3.2mm_M3, F.Cu at (29.8, 151.2)
- added H4: MountingHole, MountingHole:MountingHole_3.2mm_M3, F.Cu at (350.0, 121.4)
- added H5: MountingHole, MountingHole:MountingHole_3.2mm_M3, F.Cu at (138.1, 151.2)
- added H6: MountingHole, MountingHole:MountingHole_3.2mm_M3, F.Cu at (185.7, 54.8)
- added H7: MountingHole, MountingHole:MountingHole_3.2mm_M3, F.Cu at (290.5, 151.1)

Commit message: Added GND and other stufff.............
Parts:
- H1, H2, H3, H4, H5, H6, H7: footprint MountingHole:MountingHole_3.2mm_M3 -> MountingHole:MountingHole_2.2mm_M2_Pad_Via
- moved H2 351.1 mm to (27.4, 153.6)
- moved H5 248.4 mm to (354.8, 29.8)
- moved H6 196.5 mm to (355.5, 153.6)
- moved H4 194.4 mm to (167.4, 54.8)
- moved H3 113.2 mm to (142.4, 140.5)
- moved H7 58.0 mm to (327.0, 106.0)
- moved D79 2.38 mm to (354.8, 147.6)
- moved SW69 2.38 mm to (326.2, 123.8)
- moved SW77 2.38 mm to (307.2, 142.9)
- moved SW78 2.38 mm to (326.2, 142.9)
- moved SW79 2.38 mm to (345.3, 142.9)
- moved D69 2.38 mm to (335.8, 128.6)
- moved D77 2.38 mm to (316.7, 147.6)
- moved D78 2.38 mm to (335.8, 147.6)
- moved H1 1.65 mm to (28.1, 29.8)
Connections:
- net Net-(A1-GND-Pad13) renamed GND
Routing:
- net /COL12: track 316.8 -> 309.9 mm
- net /COL11: track 326.2 -> 320.8 mm
- net /ROW5: track 445.4 -> 442.5 mm
- net /COL14: track 93.2 -> 94.2 mm
Other:
- board size 338.1 x 133.3 mm -> 337.2 x 133 mm

Commit message: PCB should be done....
Parts:
- removed H1, H2, H3, H4, H5, H6, H7: MountingHole, MountingHole:MountingHole_2.2mm_M2_Pad_Via
- moved D14 19.1 mm to (295.3, 47.6)
- moved D69 15.1 mm to (321.5, 133.3)
- moved SW79 15.1 mm to (331.0, 147.6)
- moved SW77 15.1 mm to (292.9, 147.6)
- moved SW78 15.1 mm to (311.9, 147.6)
- moved SW69 15.0 mm to (312.0, 128.6)
- moved D77 14.7 mm to (302.4, 151.2)
- moved D78 14.7 mm to (321.5, 151.2)
- moved D79 14.7 mm to (340.5, 151.2)
- moved A1 9.86 mm to (321.2, 31.5)
Connections:
- A1 pad 1: /ROW0 -> /COL0
- A1 pad 10: /COL1 -> /COL7
- A1 pad 11: /COL2 -> /COL8
- A1 pad 12: /COL3 -> /COL9
- A1 pad 14: /COL4 -> /COL10
- A1 pad 15: /COL5 -> /COL11
- A1 pad 16: /COL6 -> /COL12
- A1 pad 17: /COL7 -> /COL13
- A1 pad 19: /COL8 -> /COL14
- A1 pad 2: /ROW1 -> /COL1
- A1 pad 20: /COL9 -> /ROW0
- A1 pad 21: /COL10 -> /ROW1
- A1 pad 22: /COL11 -> /ROW2
- A1 pad 24: /COL12 -> /ROW3
- A1 pad 25: /COL13 -> /ROW4
- A1 pad 26: /COL14 -> /ROW5
- A1 pad 4: /ROW2 -> /COL2
- A1 pad 5: /ROW3 -> /COL3
- A1 pad 6: /ROW4 -> /COL4
- A1 pad 7: /ROW5 -> /COL5
- A1 pad 9: /COL0 -> /COL6
Routing:
- net /COL13: track 195.7 -> 95.6 mm
- net /COL12: track 309.9 -> 211.8 mm
- net /COL11: track 320.8 -> 227.4 mm
- net /COL10: track 325.2 -> 235.2 mm
- net /ROW5: track 442.5 -> 375.5 mm
- net /ROW4: track 375.6 -> 328.3 mm
- net /COL8: track 301.9 -> 270.6 mm
- net /COL9: track 282.8 -> 251.9 mm
- net /ROW2: track 326.0 -> 296.1 mm
- net /COL5: track 339.5 -> 310.6 mm
- net /COL4: track 338.8 -> 310.7 mm
- net /COL3: track 353.5 -> 327.3 mm
- net /COL7: track 285.0 -> 259.4 mm
- net /COL6: track 301.6 -> 275.9 mm
- net /COL14: track 94.2 -> 70.4 mm
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Other:
- board size 337.2 x 133 mm -> 318.9 x 130.8 mm
