File: HCKeyboard/HCKeyboard.kicad_sch (KiCad schematic)
At the start: 161 parts, among them SW1 SW_Push, SW10 SW_Push, SW11 SW_Push, SW12 SW_Push, SW13 SW_Push, SW14 SW_Push, SW16 SW_Push, SW17 SW_Push, SW18 SW_Push, SW19 SW_Push, SW2 SW_Push, SW20 SW_Push, SW21 SW_Push, SW22 SW_Push, SW23 SW_Push, SW24 SW_Push, SW25 SW_Push, SW26 SW_Push, SW27 SW_Push, SW28 SW_Push, SW29 SW_Push, SW3 SW_Push, SW30 SW_Push, SW31 SW_Push, SW32 SW_Push, SW33 SW_Push, SW34 SW_Push, SW35 SW_Push, SW36 SW_Push, SW37 SW_Push, SW38 SW_Push, SW39 SW_Push, SW4 SW_Push, SW40 SW_Push, SW41 SW_Push, SW42 SW_Push, SW43 SW_Push, SW44 SW_Push, SW45 SW_Push, SW46 SW_Push, SW47 SW_Push, SW48 SW_Push, SW49 SW_Push, SW5 SW_Push, SW50 SW_Push, SW51 SW_Push, SW52 SW_Push, SW53 SW_Push, SW54 SW_Push, SW55 SW_Push, SW56 SW_Push, SW57 SW_Push, SW58 SW_Push, SW59 SW_Push, SW6 SW_Push, SW60 SW_Push, SW61 SW_Push, SW62 SW_Push, SW63 SW_Push, SW64 SW_Push, SW65 SW_Push, SW66 SW_Push, SW67 SW_Push, SW68 SW_Push, SW69 SW_Push, SW7 SW_Push, SW70 SW_Push, SW71 SW_Push, SW72 SW_Push, SW73 SW_Push, SW74 SW_Push, SW75 SW_Push, SW76 SW_Push, SW77 SW_Push, SW78 SW_Push, SW79 SW_Push, SW8 SW_Push, SW9 SW_Push

Commit message: Added mounting holes.
Parts:
- added H1, H2, H3, H4, H5, H6, H7: MountingHole, MountingHole:MountingHole_3.2mm_M3, symbol Mechanical:MountingHole

Commit message: Added GND and other stufff.............
Parts:
- H1, H2, H3, H4, H5, H6, H7: footprint MountingHole:MountingHole_3.2mm_M3 -> MountingHole:MountingHole_2.2mm_M2_Pad_Via
Connections:
- net GND: now reaches A1.13 (GND), A1.18 (GND), A1.23 (GND), A1.28 (GND), A1.3 (GND), A1.38 (GND), A1.8 (GND)
Changed lines of the file:
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@@
 			)
 		)
-		(property "Footprint" "MountingHole:MountingHole_3.2mm_M3"
+		(property "Footprint" "MountingHole:MountingHole_2.2mm_M2_Pad_Via"
 			(at 322.58 78.74 0)
 			(hide yes)
@@
 			)
 		)
-		(property "Footprint" "MountingHole:MountingHole_3.2mm_M3"
+		(property "Footprint" "MountingHole:MountingHole_2.2mm_M2_Pad_Via"
 			(at 360.68 73.66 0)
 			(hide yes)
@@
 			)
 		)
-		(property "Footprint" "MountingHole:MountingHole_3.2mm_M3"
+		(property "Footprint" "MountingHole:MountingHole_2.2mm_M2_Pad_Via"
 			(at 341.63 73.66 0)
 			(hide yes)
@@
 			)
 		)
-		(property "Footprint" "MountingHole:MountingHole_3.2mm_M3"
+		(property "Footprint" "MountingHole:MountingHole_2.2mm_M2_Pad_Via"
 			(at 322.58 73.66 0)
 			(hide yes)
@@
 			)
 		)
-		(property "Footprint" "MountingHole:MountingHole_3.2mm_M3"
+		(property "Footprint" "MountingHole:MountingHole_2.2mm_M2_Pad_Via"
 			(at 341.63 83.82 0)
 			(hide yes)
@@
 			)
 		)
-		(property "Footprint" "MountingHole:MountingHole_3.2mm_M3"
+		(property "Footprint" "MountingHole:MountingHole_2.2mm_M2_Pad_Via"
 			(at 322.58 83.82 0)
 			(hide yes)
@@
 			)
 		)
-		(property "Footprint" "MountingHole:MountingHole_3.2mm_M3"
+		(property "Footprint" "MountingHole:MountingHole_2.2mm_M2_Pad_Via"
 			(at 341.63 78.74 0)
 			(hide yes)
@@
 					(unit 1)
 				)
+			)
+		)
+	)
+	(symbol
+		(lib_id "power:GND")
+		(at 60.96 229.87 0)
+		(unit 1)
+		(body_style 1)
+		(exclude_from_sim no)
+		(in_bom yes)
+		(on_board yes)
+		(in_pos_files yes)
+		(dnp no)
+		(fields_autoplaced yes)
+		(property "Reference" "#PWR01"
+			(at 60.96 236.22 0)
+			(hide yes)
+			(show_name no)
+			(do_not_autoplace no)
+			(effects
+				(font
+					(size 1.27 1.27)
+				)
+			)
+		)
+		(property "Value" "GND"
+			(at 60.96 234.95 0)
+			(show_name no)
+			(do_not_autoplace no)
+			(effects
+				(font
+					(size 1.27 1.27)
+				)
+			)
+		)
+		(property "Footprint" ""
+			(at 60.96 229.87 0)
+			(hide yes)
+			(show_name no)
+			(do_not_autoplace no)
+			(effects
+				(font
+					(size 1.27 1.27)
+				)
+			)
+		)
+		(property "Datasheet" ""
+			(at 60.96 229.87 0)
+			(hide yes)
+			(show_name no)
+			(do_not_autoplace no)
+			(effects
+				(font
+					(size 1.27 1.27)
+				)
+			)
+		)
+		(property "Description" "Power symbol creates a global label with name \"GND\" , ground"
+			(at 60.96 229.87 0)
+			(hide yes)
+			(show_name no)
+			(do_not_autoplace no)
+			(effects
+				(font
+					(size 1.27 1.27)
+				)
+			)
+		)
+		(pin "1"
+		)
+		(instances
+			(project "HCKeyboard"
+				(path "/11e5d0eb-fed0-439e-a549-134be420093f"
+					(reference "#PWR01")
+					(unit 1)
+				)

Commit message: PCB should be done....
Parts:
- removed H1, H2, H3, H4, H5, H6, H7: MountingHole, MountingHole:MountingHole_2.2mm_M2_Pad_Via, symbol Mechanical:MountingHole
Connections:
- net COL0: now also A1.1 (GPIO0); no longer A1.9 (GPIO6)
- net COL1: now also A1.2 (GPIO1); no longer A1.10 (GPIO7)
- net COL10: now also A1.14 (GPIO10); no longer A1.21 (GPIO16)
- net COL11: now also A1.15 (GPIO11); no longer A1.22 (GPIO17)
- net COL12: now also A1.16 (GPIO12); no longer A1.24 (GPIO18)
- net COL13: now also A1.17 (GPIO13); no longer A1.25 (GPIO19)
- net COL14: now also A1.19 (GPIO14); no longer A1.26 (GPIO20)
- net COL2: now also A1.4 (GPIO2); no longer A1.11 (GPIO8)
- net COL3: now also A1.5 (GPIO3); no longer A1.12 (GPIO9)
- net COL4: now also A1.6 (GPIO4); no longer A1.14 (GPIO10)
- net COL5: now also A1.7 (GPIO5); no longer A1.15 (GPIO11)
- net COL6: now also A1.9 (GPIO6); no longer A1.16 (GPIO12)
- net COL7: now also A1.10 (GPIO7); no longer A1.17 (GPIO13)
- net COL8: now also A1.11 (GPIO8); no longer A1.19 (GPIO14)
- net COL9: now also A1.12 (GPIO9); no longer A1.20 (GPIO15)
- net ROW0: now also A1.20 (GPIO15); no longer A1.1 (GPIO0)
- net ROW1: now also A1.21 (GPIO16); no longer A1.2 (GPIO1)
- net ROW2: now also A1.22 (GPIO17); no longer A1.4 (GPIO2)
- net ROW3: now also A1.24 (GPIO18); no longer A1.5 (GPIO3)
- net ROW4: now also A1.25 (GPIO19); no longer A1.6 (GPIO4)
- net ROW5: now also A1.26 (GPIO20); no longer A1.7 (GPIO5)
